File: electronics/rc-brake-lights.kicad_pcb (KiCad board)
At the start: 2 copper layers, 22 x 10 mm, 9 parts, among them J1 TH, J2 LED, SW1 Setup button, U1 STC15W104

Commit message: Make output connector right-angle
Parts:
- C1: value 1u -> 10u
- J2: footprint Pin_Headers:Pin_Header_Straight_1x03_Pitch2.54mm -> Pin_Headers:Pin_Header_Angled_1x03_Pitch2.54mm; moved to B.Cu
- turned J2 to 0 degrees
Changed lines of the file:
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@@
     (pad_to_mask_clearance 0.1524)
     (aux_axis_origin 0 0)
-    (visible_elements FFFFFF7F)
+    (visible_elements FFFFEF7F)
     (pcbplotparams
       (layerselection 0x00030_80000001)
@@
     (add_net VCC)
   )
-  (module Pin_Headers:Pin_Header_Straight_1x03_Pitch2.54mm (layer F.Cu)
-    (at 120.098 102.54 180)
-    (descr "Through hole straight pin header, 1x03, 2.54mm pitch, single row")
-    (tags "Through hole pin header THT 1x03 2.54mm single row")
-    (fp_text reference J2 (at 2.032 -1.27 180) (layer F.SilkS) hide
-      (effects (font (size 1 1) (thickness 0.15)))
-    )
-    (fp_text value LED (at 0.032 4.699 270) (layer F.Fab)
-      (effects (font (size 1 1) (thickness 0.15)))
-    )
-    (fp_line (start -0.635 -1.27) (end 1.27 -1.27) (layer F.Fab) (width 0.1))
-    (fp_line (start 1.27 -1.27) (end 1.27 6.35) (layer F.Fab) (width 0.1))
-    (fp_line (start 1.27 6.35) (end -1.27 6.35) (layer F.Fab) (width 0.1))
-    (fp_line (start -1.27 6.35) (end -1.27 -0.635) (layer F.Fab) (width 0.1))
-    (fp_line (start -1.27 -0.635) (end -0.635 -1.27) (layer F.Fab) (width 0.1))
-    (fp_line (start -1.8 -1.8) (end -1.8 6.85) (layer F.CrtYd) (width 0.05))
-    (fp_line (start -1.8 6.85) (end 1.8 6.85) (layer F.CrtYd) (width 0.05))
-    (fp_line (start 1.8 6.85) (end 1.8 -1.8) (layer F.CrtYd) (width 0.05))
-    (fp_line (start 1.8 -1.8) (end -1.8 -1.8) (layer F.CrtYd) (width 0.05))
-    (fp_text user %R (at 0 1.397 270) (layer F.Fab)
-      (effects (font (size 1 1) (thickness 0.15)))
-    )
-    (pad 1 thru_hole rect (at 0 0 180) (size 1.7 1.7) (drill 1) (layers *.Cu *.Mask)
+  (module Pin_Headers:Pin_Header_Angled_1x03_Pitch2.54mm (layer B.Cu)
+    (at 120.098 102.54)
+    (descr "Through hole angled pin header, 1x03, 2.54mm pitch, 6mm pin length, single row")
+    (tags "Through hole angled pin header THT 1x03 2.54mm single row")
+    (fp_text reference J2 (at 4.385 2.27) (layer B.SilkS) hide
+      (effects (font (size 1 1) (thickness 0.15)) (justify mirror))
+    )
+    (fp_text value LED (at 11.982 -2.464) (layer F.Fab)
+      (effects (font (size 1 1) (thickness 0.15)))
+    )
+    (fp_line (start 2.135 1.27) (end 4.04 1.27) (layer B.Fab) (width 0.1))
+    (fp_line (start 4.04 1.27) (end 4.04 -6.35) (layer B.Fab) (width 0.1))
+    (fp_line (start 4.04 -6.35) (end 1.5 -6.35) (layer B.Fab) (width 0.1))
+    (fp_line (start 1.5 -6.35) (end 1.5 0.635) (layer B.Fab) (width 0.1))
+    (fp_line (start 1.5 0.635) (end 2.135 1.27) (layer B.Fab) (width 0.1))
+    (fp_line (start -0.32 0.32) (end 1.5 0.32) (layer B.Fab) (width 0.1))
+    (fp_line (start -0.32 0.32) (end -0.32 -0.32) (layer B.Fab) (width 0.1))
+    (fp_line (start -0.32 -0.32) (end 1.5 -0.32) (layer B.Fab) (width 0.1))
+    (fp_line (start 4.04 0.32) (end 10.04 0.32) (layer B.Fab) (width 0.1))
+    (fp_line (start 10.04 0.32) (end 10.04 -0.32) (layer B.Fab) (width 0.1))
+    (fp_line (start 4.04 -0.32) (end 10.04 -0.32) (layer B.Fab) (width 0.1))
+    (fp_line (start -0.32 -2.22) (end 1.5 -2.22) (layer B.Fab) (width 0.1))
+    (fp_line (start -0.32 -2.22) (end -0.32 -2.86) (layer B.Fab) (width 0.1))
+    (fp_line (start -0.32 -2.86) (end 1.5 -2.86) (layer B.Fab) (width 0.1))
+    (fp_line (start 4.04 -2.22) (end 10.04 -2.22) (layer B.Fab) (width 0.1))
+    (fp_line (start 10.04 -2.22) (end 10.04 -2.86) (layer B.Fab) (width 0.1))
+    (fp_line (start 4.04 -2.86) (end 10.04 -2.86) (layer B.Fab) (width 0.1))
+    (fp_line (start -0.32 -4.76) (end 1.5 -4.76) (layer B.Fab) (width 0.1))
+    (fp_line (start -0.32 -4.76) (end -0.32 -5.4) (layer B.Fab) (width 0.1))
+    (fp_line (start -0.32 -5.4) (end 1.5 -5.4) (layer B.Fab) (width 0.1))
+    (fp_line (start 4.04 -4.76) (end 10.04 -4.76) (layer B.Fab) (width 0.1))
+    (fp_line (start 10.04 -4.76) (end 10.04 -5.4) (layer B.Fab) (width 0.1))
+    (fp_line (start 4.04 -5.4) (end 10.04 -5.4) (layer B.Fab) (width 0.1))
+    (fp_line (start 1.11 -0.38) (end 1.44 -0.38) (layer B.SilkS) (width 0.12))
+    (fp_line (start 1.042929 -2.16) (end 1.44 -2.16) (layer B.SilkS) (width 0.12))
+    (fp_line (start 1.042929 -2.92) (end 1.44 -2.92) (layer B.SilkS) (width 0.12))
+    (fp_line (start -1.8 1.8) (end -1.8 -6.85) (layer B.CrtYd) (width 0.05))
+    (fp_line (start -1.8 -6.85) (end 10.55 -6.85) (layer B.CrtYd) (width 0.05))
+    (fp_line (start 10.55 -6.85) (end 10.55 1.8) (layer B.CrtYd) (width 0.05))
+    (fp_line (start 10.55 1.8) (end -1.8 1.8) (layer B.CrtYd) (width 0.05))
+    (fp_text user %R (at 2.77 -2.54 90) (layer F.Fab)
+      (effects (font (size 1 1) (thickness 0.15)))
+    )
+    (pad 1 thru_hole rect (at 0 0) (size 1.7 1.7) (drill 1) (layers *.Cu *.Mask)
       (net 2 GND))
-    (pad 2 thru_hole oval (at 0 2.54 180) (size 1.7 1.7) (drill 1) (layers *.Cu *.Mask)
+    (pad 2 thru_hole oval (at 0 -2.54) (size 1.7 1.7) (drill 1) (layers *.Cu *.Mask)
       (net 5 /Brake_LED))
-    (pad 3 thru_hole oval (at 0 5.08 180) (size 1.7 1.7) (drill 1) (layers *.Cu *.Mask)
+    (pad 3 thru_hole oval (at 0 -5.08) (size 1.7 1.7) (drill 1) (layers *.Cu *.Mask)
       (net 6 /Reverse_LED))
-    (model ${KISYS3DMOD}/Pin_Headers.3dshapes/Pin_Header_Straight_1x03_Pitch2.54mm.wrl
-      (at (xyz 0 0 0))
-      (scale (xyz 1 1 1))
-      (rotate (xyz 0 0 0))
+    (model ${KISYS3DMOD}/Pin_Headers.3dshapes/Pin_Header_Angled_1x03_Pitch2.54mm.wrl
+      (at (xyz 0 -0.2 -0.075))
+      (scale (xyz 1 1 1))
+      (rotate (xyz 180 0 0))
     )
   )
@@
       (effects (font (size 1 1) (thickness 0.15)))
     )
-    (fp_text value 1u (at 1.905 0) (layer F.Fab)
+    (fp_text value 10u (at 2.3368 0) (layer F.Fab)
       (effects (font (size 1 1) (thickness 0.15)))
     )
@@
       (effects (font (size 1 1) (thickness 0.15)))
     )
-    (fp_text value 1k (at -1.905 0 180) (layer F.Fab)
+    (fp_text value 1k (at -1.9812 0 180) (layer F.Fab)
       (effects (font (size 1 1) (thickness 0.15)))
     )
@@
       (effects (font (size 1 1) (thickness 0.15)))
     )
-    (fp_text value 1N4148 (at -2.921 0 180) (layer F.Fab)
-      (effects (font (size 0.6 0.6) (thickness 0.15)))
+    (fp_text value 1N4148 (at -4.064 0 180) (layer F.Fab)
+      (effects (font (size 1 1) (thickness 0.15)))
     )
     (fp_text user %R (at 1.27 0 270) (layer F.Fab)
@@
       (effects (font (size 1 1) (thickness 0.15)))
     )
-    (fp_text value TH (at 1.778 0 90) (layer F.Fab)
-      (effects (font (size 1 1) (thickness 0.15)))
-    )
+    (fp_text value TH (at 1.778 0 90) (layer F.Fab) hide
+      (effects (font (size 1 1) (thickness 0.15)))
+    )
